File: pcbs/null36-unrouted.kicad_pcb (KiCad board)
At the start: 2 copper layers, 123.2 x 106.1 mm, 40 parts

Commit message: v3 pcb design
Parts:
- added DISP1: , ceoloide:display_ssd1306, F.Cu at (247.0, 113.0)
- added MH1: , ceoloide:mounting_hole_npth, F.Cu at (159.5, 140.5)
- added MH2: , ceoloide:mounting_hole_npth, F.Cu at (178.5, 100.1)
- added MH3: , ceoloide:mounting_hole_npth, F.Cu at (243.1, 157.8)
- added MH4: , ceoloide:mounting_hole_npth, F.Cu at (233.5, 112.0)
- added MH5: , ceoloide:mounting_hole_npth, F.Cu at (197.5, 145.2)
- moved JST1 4.12 mm to (242.0, 139.0)
- moved PWR1 4.12 mm to (254.0, 153.2)
- moved RST1 4.01 mm to (254.0, 139.0)
- moved D1 1.00 mm to (155.7, 153.0)
- moved D10 1.00 mm to (212.7, 138.8)
- moved D11 1.00 mm to (212.7, 119.8)
- moved D12 1.00 mm to (212.7, 100.8)
- moved D13 1.00 mm to (231.7, 143.5)
- moved D14 1.00 mm to (231.7, 124.5)
- moved D15 1.00 mm to (231.7, 105.5)
- moved D16 1.00 mm to (212.7, 162.5)
- moved D2 1.00 mm to (155.7, 134.0)
- moved D3 1.00 mm to (155.7, 115.0)
- moved D4 1.00 mm to (174.7, 134.0)
- moved D5 1.00 mm to (174.7, 115.0)
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Connections:
- net far_thumb renamed far_th
- net home_thumb renamed inn_th
- net index_bottom renamed ind_bo
- net index_home renamed ind_ho
- net index_top renamed ind_to
- net inner_bottom renamed inn_bo
- net inner_home renamed inn_ho
- net inner_top renamed inn_to
- net middle_bottom renamed mi_bo
- net middle_home renamed mi_ho
- net middle_top renamed mi_to
- net near_thumb renamed ind_th
- net pinky_bottom renamed pin_bo
- net pinky_home renamed pin_ho
- net pinky_top renamed pin_to
- net ring_bottom renamed ri_bo
- net ring_home renamed ri_ho
- net ring_top renamed ri_to
- D1 pad 1: bottom -> bo
- D10 pad 1: bottom -> bo
- D11 pad 1: home -> ho
- D12 pad 1: top -> to
- D13 pad 1: bottom -> bo
- D14 pad 1: home -> ho
- D15 pad 1: top -> to
- D16 pad 1: thumb -> th
- D17 pad 1: thumb -> th
- D18 pad 1: thumb -> th
- D2 pad 1: home -> ho
- D3 pad 1: top -> to
- D4 pad 1: bottom -> bo
- D5 pad 1: home -> ho
- D6 pad 1: top -> to
- D7 pad 1: bottom -> bo
- D8 pad 1: home -> ho
- D9 pad 1: top -> to
- MCU1 pad 11: c5 -> inn
- MCU1 pad 12: c6 -> far
- MCU1 pad 13: r0 -> th
- MCU1 pad 14: c4 -> ind
- MCU1 pad 16: c2 -> mi
- MCU1 pad 17: c3 -> ri
- MCU1 pad 5: c1 -> pin
- MCU1 pad 6: r1 -> to
- MCU1 pad 7: r2 -> ho
- MCU1 pad 8: r3 -> bo
- S1 pad 2: bottom -> pin
- S10 pad 2: bottom -> ind
- S11 pad 2: home -> ind
- S12 pad 2: top -> ind
- S13 pad 2: bottom -> inn
- S14 pad 2: home -> inn
- S15 pad 2: top -> inn
- S16 pad 2: thumb -> ind
- S17 pad 2: thumb -> inn
- S18 pad 2: thumb -> far
- S2 pad 2: home -> pin
- S3 pad 2: top -> pin
- S4 pad 2: bottom -> ri
- S5 pad 2: home -> ri
- S6 pad 2: top -> ri
- S7 pad 2: bottom -> mi
- S8 pad 2: home -> mi
- S9 pad 2: top -> mi
Routing:
- net bottom: track 115.5 -> 0.00 mm, vias 5 -> 0
- net home: track 115.5 -> 0.00 mm, vias 5 -> 0
- net top: track 115.5 -> 0.00 mm, vias 5 -> 0
- net inn: track 0.00 -> 92.4 mm, vias 0 -> 4
- net ind: track 0.00 -> 92.4 mm, vias 0 -> 4
- net thumb: track 69.3 -> 0.00 mm, vias 3 -> 0
- net pin: track 0.00 -> 69.3 mm, vias 0 -> 3
- net ri: track 0.00 -> 69.3 mm, vias 0 -> 3
- net mi: track 0.00 -> 69.3 mm, vias 0 -> 3
- net far: track 0.00 -> 23.1 mm, vias 0 -> 1
- net DISP1_4: track 0.00 -> 3.50 mm
- net DISP1_3: track 0.00 -> 3.50 mm
- net DISP1_2: track 0.00 -> 3.50 mm
- net DISP1_1: track 0.00 -> 3.50 mm
Other:
- board size 123.2 x 106.1 mm -> 124.3 x 107.2 mm

Commit message: v4 pcb design
Connections:
- net CL renamed SCL
- net far_th renamed INN_THU
- net ind_bo renamed IND_BOT
- net ind_ho renamed IND_HOM
- net ind_th renamed MID_THU
- net ind_to renamed IND_TOP
- net inn_bo renamed INN_BOT
- net inn_ho renamed INN_HOM
- net inn_th renamed IND_THU
- net inn_to renamed INN_TOP
- net mi_bo renamed MID_BOT
- net mi_ho renamed MID_HOM
- net mi_to renamed MID_TOP
- net pin_bo renamed PIN_BOT
- net pin_ho renamed PIN_HOM
- net pin_to renamed PIN_TOP
- net ri_bo renamed RIN_BOT
- net ri_ho renamed RIN_HOM
- net ri_to renamed RIN_TOP
- D1 pad 1: bo -> BOT
- D10 pad 1: bo -> BOT
- D11 pad 1: ho -> HOM
- D12 pad 1: to -> TOP
- D13 pad 1: bo -> BOT
- D14 pad 1: ho -> HOM
- D15 pad 1: to -> TOP
- D16 pad 1: th -> THU
- D17 pad 1: th -> THU
- D18 pad 1: th -> THU
- D2 pad 1: ho -> HOM
- D3 pad 1: to -> TOP
- D4 pad 1: bo -> BOT
- D5 pad 1: ho -> HOM
- D6 pad 1: to -> TOP
- D7 pad 1: bo -> BOT
- D8 pad 1: ho -> HOM
- D9 pad 1: to -> TOP
- DISP1 pad 17: DA -> SDA
- DISP1 pad 27: DA -> SDA
- MCU1 pad 1: MCU1_1 -> RAW
- MCU1 pad 11: inn -> SDA
- MCU1 pad 12: far -> THU
- MCU1 pad 13: th -> BOT
- MCU1 pad 14: ind -> HOM
- MCU1 pad 15: CS -> TOP
- MCU1 pad 16: mi -> INN
- MCU1 pad 17: ri -> IND
- MCU1 pad 18: P19 -> MID
- MCU1 pad 19: P20 -> RIN
- MCU1 pad 2: MCU1_2 -> GND
- MCU1 pad 20: P21 -> PIN
- MCU1 pad 21: MCU1_21 -> GND
- MCU1 pad 22: MCU1_22 -> GND
- MCU1 pad 23: MCU1_23 -> P0
- MCU1 pad 24: MCU1_24 -> P1
- MCU1 pad 3: MCU1_3 -> RST
- MCU1 pad 4: MCU1_4 -> VCC
- MCU1 pad 5: pin -> P21
- MCU1 pad 6: to -> P20
- MCU1 pad 7: ho -> P19
- MCU1 pad 8: bo -> P18
- MCU1 pad 9: DA -> P15
- S1 pad 2: pin -> PIN
- S10 pad 2: ind -> IND
- S11 pad 2: ind -> IND
- S12 pad 2: ind -> IND
- S13 pad 2: inn -> INN
- S14 pad 2: inn -> INN
- S15 pad 2: inn -> INN
- S16 pad 2: ind -> MID
- S17 pad 2: inn -> IND
- S18 pad 2: far -> INN
- S2 pad 2: pin -> PIN
- S3 pad 2: pin -> PIN
- S4 pad 2: ri -> RIN
- S5 pad 2: ri -> RIN
- S6 pad 2: ri -> RIN
- S7 pad 2: mi -> MID
- S8 pad 2: mi -> MID
- S9 pad 2: mi -> MID
Routing:
- net (no net): track 112.6 -> 0.00 mm
- net INN: track 0.00 -> 92.4 mm, vias 0 -> 4
- net inn: track 92.4 -> 0.00 mm, vias 4 -> 0
- net IND: track 0.00 -> 92.4 mm, vias 0 -> 4
- net ind: track 92.4 -> 0.00 mm, vias 4 -> 0
- net MID: track 0.00 -> 92.4 mm, vias 0 -> 4
- net pin: track 69.3 -> 0.00 mm, vias 3 -> 0
- net PIN: track 0.00 -> 69.3 mm, vias 0 -> 3
- net ri: track 69.3 -> 0.00 mm, vias 3 -> 0
- net RIN: track 0.00 -> 69.3 mm, vias 0 -> 3
- net mi: track 69.3 -> 0.00 mm, vias 3 -> 0
- net far: track 23.1 -> 0.00 mm, vias 1 -> 0
